File: DPPM.sch (KiCad schematic (older format))
At the start: 10 parts

Commit message: Created DPPM module
Parts:
- added R6, R7: 10k, symbol Device:R
- gave numbers to parts that had none: 10
Connections:
- net labels added: V5_REG, VBAT+_UNREG
- net labels removed: V5REG5
- wire segments 34 -> 42
Changed lines of the file:
@@
 $Descr A4 11693 8268
 encoding utf-8
-Sheet 2 2
+Sheet 2 3
 Title ""
 Date ""
@@
 $EndDescr
 $Comp
-L Battery_Management:BQ24075 U?
+L Battery_Management:BQ24075 U1
 U 1 1 5D2F022F
 P 5650 2500
-F 0 "U?" H 5650 3350 50  0000 C CNN
+F 0 "U1" H 5650 3350 50  0000 C CNN
 F 1 "BQ24075" H 5650 3250 50  0000 C CNN
 F 2 "" H 5900 1950 50  0001 L CNN
@@
 $EndComp
 $Comp
-L Connector:USB_B_Micro J?
+L Connector:USB_B_Micro J2
 U 1 1 5D2F0395
 P 2200 2200
-F 0 "J?" H 2255 2667 50  0000 C CNN
+F 0 "J2" H 2255 2667 50  0000 C CNN
 F 1 "USB_B_Micro" H 2255 2576 50  0000 C CNN
 F 2 "" H 2350 2150 50  0001 C CNN
@@
 	2100 2600 2200 2600
 $Comp
-L power:GND #PWR?
+L power:GND #PWR0101
 U 1 1 5D2F047B
 P 2200 2600
-F 0 "#PWR?" H 2200 2350 50  0001 C CNN
+F 0 "#PWR0101" H 2200 2350 50  0001 C CNN
 F 1 "GND" H 2205 2427 50  0000 C CNN
 F 2 "" H 2200 2600 50  0001 C CNN
@@
 Connection ~ 2200 2600
 $Comp
-L power:VBUS #PWR?
+L power:VBUS #PWR0102
 U 1 1 5D2F0513
 P 2500 2000
-F 0 "#PWR?" H 2500 1850 50  0001 C CNN
+F 0 "#PWR0102" H 2500 1850 50  0001 C CNN
 F 1 "VBUS" H 2650 2100 50  0000 C CNN
 F 2 "" H 2500 2000 50  0001 C CNN
@@
 $EndComp
 $Comp
-L power:VBUS #PWR?
+L power:VBUS #PWR0103
 U 1 1 5D2F0545
 P 5650 1900
-F 0 "#PWR?" H 5650 1750 50  0001 C CNN
+F 0 "#PWR0103" H 5650 1750 50  0001 C CNN
 F 1 "VBUS" H 5750 1900 50  0000 C CNN
 F 2 "" H 5650 1900 50  0001 C CNN
@@
 	1    0    0    -1
 $EndComp
-Wire Wire Line
-	6250 2200 6250 2100
 Text HLabel 6700 2100 1    50   Input ~ 0
-V5REG5
+V5_REG
 Wire Wire Line
 	5550 3100 5650 3100
 $Comp
-L power:GND #PWR?
+L power:GND #PWR0104
 U 1 1 5D2F110F
 P 5650 3100
-F 0 "#PWR?" H 5650 2850 50  0001 C CNN
+F 0 "#PWR0104" H 5650 2850 50  0001 C CNN
 F 1 "GND" H 5655 2927 50  0000 C CNN
 F 2 "" H 5650 3100 50  0001 C CNN
@@
 Connection ~ 5650 3100
 $Comp
-L power:GND #PWR?
+L power:GND #PWR0105
 U 1 1 5D2F1159
-P 7500 2100
-F 0 "#PWR?" H 7500 1850 50  0001 C CNN
-F 1 "GND" H 7505 1927 50  0000 C CNN
-F 2 "" H 7500 2100 50  0001 C CNN
-F 3 "" H 7500 2100 50  0001 C CNN
-	1    7500 2100
-	1    0    0    -1
-$EndComp
-$Comp
-L Device:C C?
+P 7650 2400
+F 0 "#PWR0105" H 7650 2150 50  0001 C CNN
+F 1 "GND" H 7655 2227 50  0000 C CNN
+F 2 "" H 7650 2400 50  0001 C CNN
+F 3 "" H 7650 2400 50  0001 C CNN
+	1    7650 2400
+	1    0    0    -1
+$EndComp
+$Comp
+L Device:C C1
 U 1 1 5D2F1239
 P 7250 2100
-F 0 "C?" V 6998 2100 50  0000 C CNN
+F 0 "C1" V 6998 2100 50  0000 C CNN
 F 1 "4.7uF" V 7089 2100 50  0000 C CNN
 F 2 "" H 7288 1950 50  0001 C CNN
@@
 	0    1    1    0
 $EndComp
-Connection ~ 6250 2100
-Wire Wire Line
-	6250 2100 7100 2100
-Wire Wire Line
-	7400 2100 7500 2100
-Wire Wire Line
-	6250 2500 6250 2400
-$Comp
-L Connector:Conn_01x02_Male J?
+$Comp
+L Connector:Conn_01x02_Male J1
 U 1 1 5D2F131D
 P 2150 3450
-F 0 "J?" H 2256 3628 50  0000 C CNN
+F 0 "J1" H 2256 3628 50  0000 C CNN
 F 1 "Batt" H 2256 3537 50  0000 C CNN
 F 2 "" H 2150 3450 50  0001 C CNN
@@
 $EndComp
 $Comp
-L power:GND #PWR?
+L power:GND #PWR0106
 U 1 1 5D2F14A9
 P 2350 3550
-F 0 "#PWR?" H 2350 3300 50  0001 C CNN
+F 0 "#PWR0106" H 2350 3300 50  0001 C CNN
 F 1 "GND" H 2355 3377 50  0000 C CNN
 F 2 "" H 2350 3550 50  0001 C CNN
@@
 $EndComp
 $Comp
-L Device:C C?
+L Device:C C2
 U 1 1 5D2F14EF
 P 7250 2400
-F 0 "C?" V 6998 2400 50  0000 C CNN
-F 1 "4.7uF" V 7089 2400 50  0000 C CNN
+F 0 "C2" V 7300 2250 50  0000 C CNN
+F 1 "4.7uF" V 7400 2400 50  0000 C CNN
 F 2 "" H 7288 2250 50  0001 C CNN
 F 3 "~" H 7250 2400 50  0001 C CNN
@@
 	0    1    1    0
 $EndComp
-$Comp
-L power:GND #PWR?
-U 1 1 5D2F1511
-P 7500 2400
-F 0 "#PWR?" H 7500 2150 50  0001 C CNN
-F 1 "GND" H 7505 2227 50  0000 C CNN
-F 2 "" H 7500 2400 50  0001 C CNN
-F 3 "" H 7500 2400 50  0001 C CNN
-	1    7500 2400
-	1    0    0    -1
-$EndComp
-Wire Wire Line
-	7500 2400 7400 2400
 Wire Wire Line
 	6250 2400 6850 2400
-Connection ~ 6250 2400
-$Comp
-L Device:R R?
+$Comp
+L Device:R R5
 U 1 1 5D2F15DB
 P 6700 2600
-F 0 "R?" V 6600 2450 50  0000 C CNN
+F 0 "R5" V 6600 2450 50  0000 C CNN
 F 1 "10k" V 6584 2600 50  0000 C CNN
 F 2 "" V 6630 2600 50  0001 C CNN
@@
 Wire Wire Line
 	7400 2600 7400 2400
-Connection ~ 7400 2400
 Text HLabel 7400 2800 2    50   Input ~ 0
 \EXT_PWR_AVAIL_5V
@@
 BAT+
 Wire Wire Line
-	2850 3450 2350 3450
+	2850 3450 2600 3450
 Text Label 6850 2300 0    50   ~ 0
 BAT+
@@
 DISABLE_BATT
 $Comp
-L Device:R R?
+L Device:R R1
 U 1 1 5D2F25F0
 P 4750 1300
-F 0 "R?" V 4543 1300 50  0000 C CNN
+F 0 "R1" V 4543 1300 50  0000 C CNN
 F 1 "10k" V 4634 1300 50  0000 C CNN
 F 2 "" V 4680 1300 50  0001 C CNN
@@
 $EndComp
 $Comp
-L power:GND #PWR?
+L power:GND #PWR0108
 U 1 1 5D2F2658
 P 5200 1300
-F 0 "#PWR?" H 5200 1050 50  0001 C CNN
+F 0 "#PWR0108" H 5200 1050 50  0001 C CNN
 F 1 "GND" H 5205 1127 50  0000 C CNN
 F 2 "" H 5200 1300 50  0001 C CNN
@@
 NoConn ~ 5050 2400
 Text HLabel 4400 2600 0    50   Input ~ 0
-V5REG5
+V5_REG
 Wire Wire Line
 	4400 2600 5050 2600
 $Comp
-L power:GND #PWR?
+L power:GND #PWR0109
 U 1 1 5D2F34F1
 P 3900 3000
-F 0 "#PWR?" H 3900 2750 50  0001 C CNN
+F 0 "#PWR0109" H 3900 2750 50  0001 C CNN
 F 1 "GND" H 3905 2827 50  0000 C CNN
 F 2 "" H 3900 3000 50  0001 C CNN
@@
 	3900 2500 5050 2500
 $Comp
-L Device:R R?
+L Device:R R3
 U 1 1 5D2F387E
 P 4750 2800
-F 0 "R?" V 4650 2650 50  0000 C CNN
+F 0 "R3" V 4650 2650 50  0000 C CNN
 F 1 "1.18k" V 4634 2800 50  0000 C CNN
 F 2 "" V 4680 2800 50  0001 C CNN
@@
 	3900 2800 3900 2500
 $Comp
-L Device:R R?
+L Device:R R4
 U 1 1 5D2F44ED
 P 4750 2900
-F 0 "R?" V 4850 2750 50  0000 C CNN
+F 0 "R4" V 4850 2750 50  0000 C CNN
 F 1 "1.13k" V 4850 2900 50  0000 C CNN
 F 2 "" V 4680 2900 50  0001 C CNN
@@
 \CHG_ENABLE
 $Comp
-L Device:R R?
+L Device:R R2
 U 1 1 5D2F52D4
 P 4750 1500
-F 0 "R?" V 4850 1350 50  0000 C CNN
+F 0 "R2" V 4850 1350 50  0000 C CNN
 F 1 "10k" V 4850 1500 50  0000 C CNN
 F 2 "" V 4680 1500 50  0001 C CNN
@@
 Wire Wire Line
 	5000 1300 4900 1300
+Wire Wire Line
+	6250 2100 7100 2100
+Wire Wire Line
+	6250 2200 6250 2100
+Connection ~ 6250 2100
+Wire Wire Line
+	6250 2500 6250 2400
+Connection ~ 6250 2400
+Text HLabel 7250 1300 0    50   Input ~ 0
+\EXT_PWR_AVAIL_5V
+Text HLabel 7250 1450 0    50   Input ~ 0
+\BATT_CHGNG_5V
+$Comp
+L Device:R R6
+U 1 1 5D2FB49A
+P 7600 1300
+F 0 "R6" V 7393 1300 50  0000 C CNN
+F 1 "10k" V 7484 1300 50  0000 C CNN
+F 2 "" V 7530 1300 50  0001 C CNN
+F 3 "~" H 7600 1300 50  0001 C CNN
+	1    7600 1300
+	0    1    1    0
+$EndComp
+Wire Wire Line
+	7450 1300 7250 1300
+$Comp
+L Device:R R7
+U 1 1 5D2FBBDF
+P 7600 1450
+F 0 "R7" V 7700 1350 50  0000 C CNN
+F 1 "10k" V 7700 1450 50  0000 C CNN
+F 2 "" V 7530 1450 50  0001 C CNN
+F 3 "~" H 7600 1450 50  0001 C CNN
+	1    7600 1450
+	0    1    1    0
+$EndComp
+Wire Wire Line
+	7450 1450 7250 1450
+Wire Wire Line
+	7750 1450 7750 1300
+Wire Wire Line
+	8450 1300 8450 1200
+Wire Wire Line
+	7750 1300 8450 1300
+Connection ~ 7750 1300
+Text HLabel 8450 1200 1    50   Input ~ 0
+V5_REG
+Wire Wire Line
+	7400 2400 7650 2400
+Connection ~ 7400 2400
+Wire Wire Line
+	7400 2100 7400 2400
+Text HLabel 2850 3200 2    50   Input ~ 0
+VBAT+_UNREG
+Wire Wire Line
+	2850 3200 2600 3200
+Wire Wire Line
+	2600 3200 2600 3450
+Connection ~ 2600 3450
+Wire Wire Line
+	2600 3450 2350 3450
 $EndSCHEMATC
