File: _saved_launch-device-hurestic.sch (KiCad schematic (older format))
At the start: 2 parts

Commit message: Created DPPM module
Parts:
- added S?: 1825232-1, 18252321, symbol SamacSys_Parts:1825232-1
Connections:
- wire segments 2 -> 7
Other:
- moved on the sheet: U?
Changed lines of the file:
@@
 F6 "\\CHG_ENABLE" I R 9900 1800 50
 F7 "VBAT+_UNREG" I L 8700 1550 50
-F8 "V5_REG" I L 8700 1800 50
+F8 "V5_REG" I L 8700 1450 50
 $EndSheet
 $Comp
@@
 L Regulator_Linear:LM1117-3.3 U?
 U 1 1 5D300A86
-P 6200 1600
-F 0 "U?" V 6154 1705 50  0000 L CNN
-F 1 "LM1117-3.3" V 6245 1705 50  0000 L CNN
-F 2 "" H 6200 1600 50  0001 C CNN
-F 3 "http://www.ti.com/lit/ds/symlink/lm1117.pdf" H 6200 1600 50  0001 C CNN
-	1    6200 1600
+P 6200 2050
+F 0 "U?" V 6154 2155 50  0000 L CNN
+F 1 "LM1117-3.3" V 6245 2155 50  0000 L CNN
+F 2 "" H 6200 2050 50  0001 C CNN
+F 3 "http://www.ti.com/lit/ds/symlink/lm1117.pdf" H 6200 2050 50  0001 C CNN
+	1    6200 2050
 	0    1    1    0
 $EndComp
@@
 L power:GND #PWR?
 U 1 1 5D301560
-P 5700 1600
-F 0 "#PWR?" H 5700 1350 50  0001 C CNN
-F 1 "GND" H 5705 1427 50  0000 C CNN
-F 2 "" H 5700 1600 50  0001 C CNN
-F 3 "" H 5700 1600 50  0001 C CNN
-	1    5700 1600
+P 5700 2050
+F 0 "#PWR?" H 5700 1800 50  0001 C CNN
+F 1 "GND" H 5705 1877 50  0000 C CNN
+F 2 "" H 5700 2050 50  0001 C CNN
+F 3 "" H 5700 2050 50  0001 C CNN
+	1    5700 2050
 	1    0    0    -1
 $EndComp
 Wire Wire Line
-	5700 1600 5900 1600
+	5700 2050 5900 2050
 $Comp
 L power:GND #PWR?
@@
 Wire Wire Line
 	8300 1650 8700 1650
+$Comp
+L SamacSys_Parts:1825232-1 S?
+U 1 1 5D30633E
+P 7400 1600
+F 0 "S?" V 7896 1272 50  0000 R CNN
+F 1 "1825232-1" V 7805 1272 50  0000 R CNN
+F 2 "18252321" H 8150 1700 50  0001 L CNN
+F 3 "https://componentsearchengine.com/Datasheets/1/1825232-1.pdf" H 8150 1600 50  0001 L CNN
+F 4 "TE CONNECTIVITY - 1825232-1 - SLIDE SWITCH, SPDT, 0.2A, 30VDC, SOLDER" H 8150 1500 50  0001 L CNN "Description"
+F 5 "3.7" H 8150 1400 50  0001 L CNN "Height"
+F 6 "655-1825232-1" H 8150 1300 50  0001 L CNN "Mouser Part Number"
+F 7 "https://www.mouser.com/Search/Refine.aspx?Keyword=655-1825232-1" H 8150 1200 50  0001 L CNN "Mouser Price/Stock"
+F 8 "TE Connectivity" H 8150 1100 50  0001 L CNN "Manufacturer_Name"
+F 9 "1825232-1" H 8150 1000 50  0001 L CNN "Manufacturer_Part_Number"
+	1    7400 1600
+	0    -1   -1   0
+$EndComp
+Wire Wire Line
+	8700 1450 8000 1450
+Wire Wire Line
+	8000 1450 8000 1600
+Wire Wire Line
+	8000 1600 7600 1600
+Wire Wire Line
+	7500 1600 7500 1750
+Wire Wire Line
+	7500 1750 6200 1750
 $EndSCHEMATC
